File: 13-Chapter/KICAD/LogicAnalizer.kicad_sch (KiCad schematic)
At the start: 102 parts, among them J1 Conn_02x01, J2 Conn_02x08_Odd_Even, J3 Conn_02x08_Odd_Even, J4 Conn_02x08_Odd_Even, J5 Conn_02x08_Odd_Even, J6 Conn_02x08_Odd_Even, J7 Conn_02x08_Odd_Even, J8 Conn_02x08_Odd_Even, J9 Conn_02x08_Odd_Even, U1 74HC164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

Commit message: Add pdf
Other:
- title: (none) -> "THOR" Digital Circuit Tester
Changed lines of the file:
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@@
 	(generator_version "8.0")
 	(paper "A3")
+	(title_block
+		(title "\"THOR\" Digital Circuit Tester")
+		(date "2024-04-14")
+	)
 	(junction
 		(at 309.88 130.81)
